Commit message: this is anti-deletion measure

File: deform/src/geo/cube_obj/cube_10_6_6.urdf (robot description, URDF)
Before this commit: robot cube_10_6_6, 1 links, 0 joints
Links:
- link baseLink: geometry collision mesh filename=cube_10_6_6.obj scale=.1 .1 .1; visual mesh filename=cube_10_6_6.obj scale=.1 .1 .1
